File: PCB/LDOA/LDOA/LDOA.sch (KiCad schematic (older format))
At the start: 20 parts, among them Q1 BC547, Q2 BC547, Q3 BC557, Q4 BC547, Q5 BC557, Q6 BC547, Q7 2N7000, Q8 IRF9520

Commit message: Se acomodaron componentes en el PCB del circuito LDOA, También se agregó el foldback. Todavía falta sumar el UVLO OVLO, y poner los bornes para entradas y salidas del circuito.
Parts:
- added C2: C, Capacitor_THT:CP_Radial_D17.0mm_P7.50mm, symbol Device:C
- added Q10, Q9: BS250, Package_TO_SOT_THT:TO-92_Inline, symbol Transistor_FET:BS250
- added R12, R13, R14, R15, R16, R17, R18, R19, R20, R21, R22, R23, R24, R25, R26: R, Resistor_THT:R_Axial_DIN0207_L6.3mm_D2.5mm_P10.16mm_Horizontal, symbol Device:R
- added U1, U2, U3: TL084, symbol Amplifier_Operational:TL084
Connections:
- net VA: now also R14.1
- net Vf: now also R20.1; no longer Q2.2 (B)
- net Vref: now also R12.2
- net VREG: now reaches Q8.3, R1.1, R3.1, R7.1
- net VREG: now also Q10.3 (S), Q9.3 (S)
- net at C1.2, Q5.1 (C), Q6.1 (C)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: now also Q10.1 (D), Q9.1 (D)
- net GND: now reaches Q7.1 (S), R10.2, R2.1, R5.1
- net GND: now also R15.2, R16.1, R18.1, R24.2
- net at C1.1, Q8.2, R11.2: now also R13.1
- new net: R14.2, R17.1, U1.2 (-)
- new net: R13.2, R16.2, U1.3 (+)
- new net: R18.2, R21.1, U2.2 (-)
- new net: R19.2, R20.2, U2.3 (+)
- new net: R12.1, R15.1, R19.1
- new net: R22.2, R25.1, R26.1, U3.2 (-)
- new net: R23.2, R24.1, U3.3 (+)
- new net: C2.2, R25.2
- new net ENLDO: Q9.2 (G)
- new net Vact: C2.1, Q10.2 (G), R26.2, U3.1
- new net Vref2: R21.2, R23.1, U2.1
- new net Vsens: R17.2, R22.1, U1.1
Other:
- note added: "Amplificador de error"
- note added: "Sensado de corriente\n"
- note added: "Sumador"
- moved on the sheet: Q8, R11
